Commit message: Milestone 2 simulation upgrade

File: src/rss_description/urdf/turtlebot3_waffle_pi_px100_arm.urdf.xacro (robot description, xacro)
@@ -1,4 +1,5 @@
 <?xml version="1.0" ?>
-<robot name="turtlebot3_waffle_pi_for_open_manipulator" xmlns:xacro="http://ros.org/wiki/xacro">
+<robot name="turtlebot3_waffle_pi"
+  xmlns:xacro="http://ros.org/wiki/xacro">
   <xacro:include filename="$(find rss_description)/urdf/common_properties.xacro"/>
   <xacro:include filename="$(find rss_description)/urdf/turtlebot3_waffle_pi.gazebo.xacro"/>
@@ -13,5 +14,5 @@
       <origin xyz="-0.064 0 0.0" rpy="0 0 0"/>
       <geometry>
-        <mesh filename="package://rss_description/meshes/bases/waffle_pi_base_for_open_manipulator.stl" scale="0.001 0.001 0.001"/>
+        <mesh filename="package://rss_description/meshes/bases/waffle_pi_base.stl" scale="0.001 0.001 0.001"/>
       </geometry>
       <material name="light_black"/>
@@ -25,8 +26,7 @@
     <inertial>
       <origin xyz="0 0 0" rpy="0 0 0"/>
-      <mass value="1.3729096e+00"/>
-      <inertia ixx="8.7002718e-03" ixy="-4.7576583e-05" ixz="1.1160499e-04"
-               iyy="8.6195418e-03" iyz="-3.5422299e-06"
-               izz="1.4612727e-02" />
+      <mass value="1.3729096e+01"/>
+      <!-- <inertia ixx="8.7002718e+01" ixy="-4.7576583e-04" ixz="1.1160499e-05" iyy="8.6195418e-02" iyz="-3.5422299e-05" izz="1.4612727e-05" /> -->
+      <inertia ixx="1e02" ixy="1e-10" ixz="1e-10" iyy="1e-3" iyz="1e-10" izz="-1e-3" />
     </inertial>
   </link>
@@ -54,8 +54,6 @@
       <origin xyz="0 0 0" />
       <mass value="2.8498940e-02" />
-      <inertia ixx="1.1175580e-05" ixy="-4.2369783e-11" ixz="-5.9381719e-09"
-               iyy="1.1192413e-05" iyz="-1.4400107e-11"
-               izz="2.0712558e-05" />
-      </inertial>
+      <inertia ixx="1.1175580e-05" ixy="-4.2369783e-11" ixz="-5.9381719e-09" iyy="1.1192413e-05" iyz="-1.4400107e-11" izz="2.0712558e-05" />
+    </inertial>
   </link>
   <joint name="wheel_right_joint" type="continuous">
@@ -74,5 +72,5 @@
     </visual>
     <collision>
-      <origin xyz="0 0.001 0" rpy="0 0 0"/>
+      <origin xyz="0 0 0" rpy="0 0 0"/>
       <geometry>
         <cylinder length="0.018" radius="0.033"/>
@@ -82,8 +80,6 @@
       <origin xyz="0 0 0" />
       <mass value="2.8498940e-02" />
-      <inertia ixx="1.1175580e-05" ixy="-4.2369783e-11" ixz="-5.9381719e-09"
-               iyy="1.1192413e-05" iyz="-1.4400107e-11"
-               izz="2.0712558e-05" />
-      </inertial>
+      <inertia ixx="1.1175580e-05" ixy="-4.2369783e-11" ixz="-5.9381719e-09" iyy="1.1192413e-05" iyz="-1.4400107e-11" izz="2.0712558e-05" />
+    </inertial>
   </link>
   <joint name="caster_back_right_joint" type="fixed">
@@ -102,7 +98,5 @@
       <origin xyz="0 0 0" />
       <mass value="0.005" />
-      <inertia ixx="0.001" ixy="0.0" ixz="0.0"
-               iyy="0.001" iyz="0.0"
-               izz="0.001" />
+      <inertia ixx="0.001" ixy="0.0" ixz="0.0" iyy="0.001" iyz="0.0" izz="0.001" />
     </inertial>
   </link>
@@ -122,7 +116,5 @@
       <origin xyz="0 0 0" />
       <mass value="0.005" />
-      <inertia ixx="0.001" ixy="0.0" ixz="0.0"
-               iyy="0.001" iyz="0.0"
-               izz="0.001" />
+      <inertia ixx="0.001" ixy="0.0" ixz="0.0" iyy="0.001" iyz="0.0" izz="0.001" />
     </inertial>
   </link>
@@ -136,5 +128,5 @@
     <parent link="base_link"/>
     <child link="base_scan"/>
-    <origin xyz="-0.024 0 0.122" rpy="0 0 0"/>
+    <origin xyz="-0.064 0 0.122" rpy="0 0 0"/>
   </joint>
   <link name="base_scan">
@@ -149,5 +141,5 @@
       <origin xyz="0.015 0 -0.0065" rpy="0 0 0"/>
       <geometry>
-        <cylinder length="0.0315" radius="0.045"/>
+        <cylinder length="0.0315" radius="0.055"/>
       </geometry>
     </collision>
@@ -155,33 +147,16 @@
       <mass value="0.114" />
       <origin xyz="0 0 0" />
-      <inertia ixx="0.001" ixy="0.0" ixz="0.0"
-               iyy="0.001" iyz="0.0"
-               izz="0.001" />
+      <inertia ixx="0.001" ixy="0.0" ixz="0.0" iyy="0.001" iyz="0.0" izz="0.001" />
     </inertial>
   </link>
-  <joint name="camera_joint" type="fixed">
-    <origin xyz="0.073 -0.011 0.084" rpy="0 0 0"/>
+  <!-- NOW START ARM !!-->
+  <!-- Include arm with joint -->
+  <joint name="fixed" type="fixed">
     <parent link="base_link"/>
-    <child link="camera_link"/>
+    <child link="arm_base_link"/>
+    <origin xyz="-0.05 0 0.14" rpy="0 0 0"/>
   </joint>
-  <link name="camera_link">
-    <collision>
-      <origin xyz="0.005 0.011 0.013" rpy="0 0 0"/>
-      <geometry>
-        <box size="0.015 0.030 0.027"/>
-      </geometry>
-    </collision>
-  </link>
-  <joint name="camera_rgb_joint" type="fixed">
-    <origin xyz="0.003 0.011 0.009" rpy="0 0 0"/>
-    <parent link="camera_link"/>
-    <child link="camera_rgb_frame"/>
-  </joint>
-  <link name="camera_rgb_frame"/>
-  <joint name="camera_rgb_optical_joint" type="fixed">
-    <origin xyz="0 0 0" rpy="-1.57 0 -1.57"/>
-    <parent link="camera_rgb_frame"/>
-    <child link="camera_rgb_optical_frame"/>
-  </joint>
-  <link name="camera_rgb_optical_frame"/>
+  <xacro:include filename="$(find rss_description)/urdf/px100.urdf.xacro">
+    <xacro:arg name="moveit" value="false"/>
+  </xacro:include>
 </robot>
